Commit message: Complete redesign: URDF, world, controllers, launch files, and Python nodes

File: color_sorting_arm/urdf/arm.gazebo.xacro (robot description, xacro)
@@ -12,29 +12,41 @@
   <!-- Gazebo materials -->
   <gazebo reference="base_link">
-    <material>Gazebo/Grey</material>
+    <material>Gazebo/DarkGrey</material>
+    <mu1>1.0</mu1>
+    <mu2>1.0</mu2>
   </gazebo>
   <gazebo reference="link1">
+    <material>Gazebo/Orange</material>
+  </gazebo>
+  <gazebo reference="link2">
     <material>Gazebo/Blue</material>
   </gazebo>
-  <gazebo reference="link2">
+  <gazebo reference="link3">
     <material>Gazebo/White</material>
   </gazebo>
-  <gazebo reference="link3">
+  <gazebo reference="link4">
     <material>Gazebo/Blue</material>
   </gazebo>
-  <gazebo reference="link4">
+  <gazebo reference="link5">
     <material>Gazebo/White</material>
-  </gazebo>
-  <gazebo reference="link5">
-    <material>Gazebo/Blue</material>
   </gazebo>
   <gazebo reference="gripper_base">
     <material>Gazebo/Grey</material>
   </gazebo>
-  <gazebo reference="gripper_left_finger">
-    <material>Gazebo/Black</material>
+  <gazebo reference="gripper_left">
+    <material>Gazebo/DarkGrey</material>
+    <mu1>1.5</mu1>
+    <mu2>1.5</mu2>
   </gazebo>
-  <gazebo reference="gripper_right_finger">
-    <material>Gazebo/Black</material>
+  <gazebo reference="gripper_right">
+    <material>Gazebo/DarkGrey</material>
+    <mu1>1.5</mu1>
+    <mu2>1.5</mu2>
+  </gazebo>
+  <gazebo reference="camera_pole">
+    <material>Gazebo/Grey</material>
+  </gazebo>
+  <gazebo reference="camera_link">
+    <material>Gazebo/DarkGrey</material>
   </gazebo>
   <!-- Camera sensor plugin -->

File: color_sorting_arm/urdf/arm.urdf.xacro (robot description, xacro)
@@ -1,56 +1,62 @@
 <?xml version="1.0"?>
 <robot xmlns:xacro="http://www.ros.org/wiki/xacro" name="sorting_arm">
-  <!-- Constants -->
+  <!-- ===================== CONSTANTS ===================== -->
   <xacro:property name="PI" value="3.1415926535897931"/>
-  <!-- Material colors -->
+  <!-- ===================== MATERIALS ===================== -->
   <material name="blue">
-    <color rgba="0 0 0.8 1"/>
-  </material>
-  <material name="black">
-    <color rgba="0 0 0 1"/>
+    <color rgba="0.2 0.4 0.8 1"/>
   </material>
   <material name="white">
-    <color rgba="1 1 1 1"/>
+    <color rgba="0.9 0.9 0.9 1"/>
   </material>
   <material name="grey">
     <color rgba="0.5 0.5 0.5 1"/>
   </material>
-  <!-- Base Link -->
+  <material name="dark_grey">
+    <color rgba="0.2 0.2 0.2 1"/>
+  </material>
+  <material name="orange">
+    <color rgba="1.0 0.5 0.0 1"/>
+  </material>
+  <!-- ===================== BASE LINK ===================== -->
   <link name="base_link">
     <visual>
-      <geometry>
-        <cylinder radius="0.1" length="0.05"/>
-      </geometry>
-      <material name="grey"/>
-    </visual>
-    <collision>
-      <geometry>
-        <cylinder radius="0.1" length="0.05"/>
-      </geometry>
-    </collision>
-    <inertial>
-      <mass value="1.0"/>
-      <inertia ixx="0.001" ixy="0.0" ixz="0.0" iyy="0.001" iyz="0.0" izz="0.001"/>
-    </inertial>
-  </link>
-  <!-- Link 1 (Rotating Base) -->
+      <origin xyz="0 0 0.025" rpy="0 0 0"/>
+      <geometry>
+        <cylinder radius="0.08" length="0.05"/>
+      </geometry>
+      <material name="dark_grey"/>
+    </visual>
+    <collision>
+      <origin xyz="0 0 0.025" rpy="0 0 0"/>
+      <geometry>
+        <cylinder radius="0.08" length="0.05"/>
+      </geometry>
+    </collision>
+    <inertial>
+      <origin xyz="0 0 0.025" rpy="0 0 0"/>
+      <mass value="2.0"/>
+      <inertia ixx="0.005" ixy="0" ixz="0" iyy="0.005" iyz="0" izz="0.005"/>
+    </inertial>
+  </link>
+  <!-- ===================== LINK 1 - ROTATING BASE ===================== -->
   <link name="link1">
     <visual>
-      <origin xyz="0 0 0.1" rpy="0 0 0"/>
-      <geometry>
-        <cylinder radius="0.05" length="0.2"/>
-      </geometry>
-      <material name="blue"/>
-    </visual>
-    <collision>
-      <origin xyz="0 0 0.1" rpy="0 0 0"/>
-      <geometry>
-        <cylinder radius="0.05" length="0.2"/>
-      </geometry>
-    </collision>
-    <inertial>
-      <origin xyz="0 0 0.1" rpy="0 0 0"/>
+      <origin xyz="0 0 0.04" rpy="0 0 0"/>
+      <geometry>
+        <cylinder radius="0.045" length="0.08"/>
+      </geometry>
+      <material name="orange"/>
+    </visual>
+    <collision>
+      <origin xyz="0 0 0.04" rpy="0 0 0"/>
+      <geometry>
+        <cylinder radius="0.045" length="0.08"/>
+      </geometry>
+    </collision>
+    <inertial>
+      <origin xyz="0 0 0.04" rpy="0 0 0"/>
       <mass value="0.5"/>
-      <inertia ixx="0.002" ixy="0.0" ixz="0.0" iyy="0.002" iyz="0.0" izz="0.0005"/>
+      <inertia ixx="0.001" ixy="0" ixz="0" iyy="0.001" iyz="0" izz="0.0005"/>
     </inertial>
   </link>
@@ -58,28 +64,28 @@
     <parent link="base_link"/>
     <child link="link1"/>
-    <origin xyz="0 0 0.025" rpy="0 0 0"/>
+    <origin xyz="0 0 0.05" rpy="0 0 0"/>
     <axis xyz="0 0 1"/>
-    <limit lower="${-PI}" upper="${PI}" effort="100" velocity="1.0"/>
-    <dynamics damping="0.7"/>
-  </joint>
-  <!-- Link 2 (Shoulder) -->
+    <limit lower="${-PI}" upper="${PI}" effort="30" velocity="1.5"/>
+    <dynamics damping="0.5" friction="0.1"/>
+  </joint>
+  <!-- ===================== LINK 2 - SHOULDER ===================== -->
   <link name="link2">
     <visual>
-      <origin xyz="0 0 0.15" rpy="0 0 0"/>
-      <geometry>
-        <box size="0.05 0.05 0.3"/>
-      </geometry>
-      <material name="white"/>
-    </visual>
-    <collision>
-      <origin xyz="0 0 0.15" rpy="0 0 0"/>
-      <geometry>
-        <box size="0.05 0.05 0.3"/>
-      </geometry>
-    </collision>
-    <inertial>
-      <origin xyz="0 0 0.15" rpy="0 0 0"/>
+      <origin xyz="0 0 0.075" rpy="0 0 0"/>
+      <geometry>
+        <box size="0.05 0.05 0.15"/>
+      </geometry>
+      <material name="blue"/>
+    </visual>
+    <collision>
+      <origin xyz="0 0 0.075" rpy="0 0 0"/>
+      <geometry>
+        <box size="0.05 0.05 0.15"/>
+      </geometry>
+    </collision>
+    <inertial>
+      <origin xyz="0 0 0.075" rpy="0 0 0"/>
       <mass value="0.4"/>
-      <inertia ixx="0.003" ixy="0.0" ixz="0.0" iyy="0.003" iyz="0.0" izz="0.0004"/>
+      <inertia ixx="0.001" ixy="0" ixz="0" iyy="0.001" iyz="0" izz="0.0003"/>
     </inertial>
   </link>
@@ -87,28 +93,28 @@
     <parent link="link1"/>
     <child link="link2"/>
-    <origin xyz="0 0 0.2" rpy="0 0 0"/>
+    <origin xyz="0 0 0.08" rpy="0 0 0"/>
     <axis xyz="0 1 0"/>
-    <limit lower="${-PI/2}" upper="${PI/2}" effort="100" velocity="1.0"/>
-    <dynamics damping="0.7"/>
-  </joint>
-  <!-- Link 3 (Elbow) -->
+    <limit lower="${-PI/2}" upper="${PI/2}" effort="30" velocity="1.5"/>
+    <dynamics damping="0.5" friction="0.1"/>
+  </joint>
+  <!-- ===================== LINK 3 - ELBOW ===================== -->
   <link name="link3">
     <visual>
-      <origin xyz="0 0 0.15" rpy="0 0 0"/>
-      <geometry>
-        <box size="0.04 0.04 0.3"/>
-      </geometry>
-      <material name="blue"/>
-    </visual>
-    <collision>
-      <origin xyz="0 0 0.15" rpy="0 0 0"/>
-      <geometry>
-        <box size="0.04 0.04 0.3"/>
-      </geometry>
-    </collision>
-    <inertial>
-      <origin xyz="0 0 0.15" rpy="0 0 0"/>
+      <origin xyz="0 0 0.075" rpy="0 0 0"/>
+      <geometry>
+        <box size="0.04 0.04 0.15"/>
+      </geometry>
+      <material name="white"/>
+    </visual>
+    <collision>
+      <origin xyz="0 0 0.075" rpy="0 0 0"/>
+      <geometry>
+        <box size="0.04 0.04 0.15"/>
+      </geometry>
+    </collision>
+    <inertial>
+      <origin xyz="0 0 0.075" rpy="0 0 0"/>
       <mass value="0.3"/>
-      <inertia ixx="0.0025" ixy="0.0" ixz="0.0" iyy="0.0025" iyz="0.0" izz="0.0003"/>
+      <inertia ixx="0.0008" ixy="0" ixz="0" iyy="0.0008" iyz="0" izz="0.0002"/>
     </inertial>
   </link>
@@ -116,28 +122,28 @@
     <parent link="link2"/>
     <child link="link3"/>
-    <origin xyz="0 0 0.3" rpy="0 0 0"/>
+    <origin xyz="0 0 0.15" rpy="0 0 0"/>
     <axis xyz="0 1 0"/>
-    <limit lower="${-PI/2}" upper="${PI/2}" effort="100" velocity="1.0"/>
-    <dynamics damping="0.7"/>
-  </joint>
-  <!-- Link 4 (Wrist Pitch) -->
+    <limit lower="${-2.5}" upper="${2.5}" effort="20" velocity="1.5"/>
+    <dynamics damping="0.3" friction="0.1"/>
+  </joint>
+  <!-- ===================== LINK 4 - WRIST PITCH ===================== -->
   <link name="link4">
     <visual>
-      <origin xyz="0 0 0.1" rpy="0 0 0"/>
-      <geometry>
-        <box size="0.03 0.03 0.2"/>
-      </geometry>
-      <material name="white"/>
-    </visual>
-    <collision>
-      <origin xyz="0 0 0.1" rpy="0 0 0"/>
-      <geometry>
-        <box size="0.03 0.03 0.2"/>
-      </geometry>
-    </collision>
-    <inertial>
-      <origin xyz="0 0 0.1" rpy="0 0 0"/>
-      <mass value="0.2"/>
-      <inertia ixx="0.001" ixy="0.0" ixz="0.0" iyy="0.001" iyz="0.0" izz="0.0002"/>
+      <origin xyz="0 0 0.04" rpy="0 0 0"/>
+      <geometry>
+        <box size="0.035 0.035 0.08"/>
+      </geometry>
+      <material name="blue"/>
+    </visual>
+    <collision>
+      <origin xyz="0 0 0.04" rpy="0 0 0"/>
+      <geometry>
+        <box size="0.035 0.035 0.08"/>
+      </geometry>
+    </collision>
+    <inertial>
+      <origin xyz="0 0 0.04" rpy="0 0 0"/>
+      <mass value="0.15"/>
+      <inertia ixx="0.0003" ixy="0" ixz="0" iyy="0.0003" iyz="0" izz="0.0001"/>
     </inertial>
   </link>
@@ -145,28 +151,28 @@
     <parent link="link3"/>
     <child link="link4"/>
-    <origin xyz="0 0 0.3" rpy="0 0 0"/>
+    <origin xyz="0 0 0.15" rpy="0 0 0"/>
     <axis xyz="0 1 0"/>
-    <limit lower="${-PI/2}" upper="${PI/2}" effort="50" velocity="1.0"/>
-    <dynamics damping="0.5"/>
-  </joint>
-  <!-- Link 5 (Wrist Roll) -->
+    <limit lower="${-PI/2}" upper="${PI/2}" effort="10" velocity="2.0"/>
+    <dynamics damping="0.2" friction="0.05"/>
+  </joint>
+  <!-- ===================== LINK 5 - WRIST ROLL ===================== -->
   <link name="link5">
     <visual>
-      <origin xyz="0 0 0.05" rpy="0 0 0"/>
-      <geometry>
-        <cylinder radius="0.025" length="0.1"/>
-      </geometry>
-      <material name="blue"/>
-    </visual>
-    <collision>
-      <origin xyz="0 0 0.05" rpy="0 0 0"/>
-      <geometry>
-        <cylinder radius="0.025" length="0.1"/>
-      </geometry>
-    </collision>
-    <inertial>
-      <origin xyz="0 0 0.05" rpy="0 0 0"/>
-      <mass value="0.1"/>
-      <inertia ixx="0.0005" ixy="0.0" ixz="0.0" iyy="0.0005" iyz="0.0" izz="0.0001"/>
+      <origin xyz="0 0 0.02" rpy="0 0 0"/>
+      <geometry>
+        <cylinder radius="0.02" length="0.04"/>
+      </geometry>
+      <material name="white"/>
+    </visual>
+    <collision>
+      <origin xyz="0 0 0.02" rpy="0 0 0"/>
+      <geometry>
+        <cylinder radius="0.02" length="0.04"/>
+      </geometry>
+    </collision>
+    <inertial>
+      <origin xyz="0 0 0.02" rpy="0 0 0"/>
+      <mass value="0.08"/>
+      <inertia ixx="0.00005" ixy="0" ixz="0" iyy="0.00005" iyz="0" izz="0.00002"/>
     </inertial>
   </link>
@@ -174,28 +180,28 @@
     <parent link="link4"/>
     <child link="link5"/>
-    <origin xyz="0 0 0.2" rpy="0 0 0"/>
+    <origin xyz="0 0 0.08" rpy="0 0 0"/>
     <axis xyz="0 0 1"/>
-    <limit lower="${-PI}" upper="${PI}" effort="50" velocity="1.0"/>
-    <dynamics damping="0.5"/>
-  </joint>
-  <!-- Gripper Base -->
+    <limit lower="${-PI}" upper="${PI}" effort="5" velocity="2.0"/>
+    <dynamics damping="0.1" friction="0.05"/>
+  </joint>
+  <!-- ===================== GRIPPER BASE ===================== -->
   <link name="gripper_base">
     <visual>
-      <origin xyz="0 0 0.02" rpy="0 0 0"/>
-      <geometry>
-        <box size="0.04 0.06 0.04"/>
+      <origin xyz="0 0 0.015" rpy="0 0 0"/>
+      <geometry>
+        <box size="0.03 0.06 0.03"/>
       </geometry>
       <material name="grey"/>
     </visual>
     <collision>
-      <origin xyz="0 0 0.02" rpy="0 0 0"/>
-      <geometry>
-        <box size="0.04 0.06 0.04"/>
-      </geometry>
-    </collision>
-    <inertial>
-      <origin xyz="0 0 0.02" rpy="0 0 0"/>
+      <origin xyz="0 0 0.015" rpy="0 0 0"/>
+      <geometry>
+        <box size="0.03 0.06 0.03"/>
+      </geometry>
+    </collision>
+    <inertial>
+      <origin xyz="0 0 0.015" rpy="0 0 0"/>
       <mass value="0.05"/>
-      <inertia ixx="0.0001" ixy="0.0" ixz="0.0" iyy="0.0001" iyz="0.0" izz="0.0001"/>
+      <inertia ixx="0.00002" ixy="0" ixz="0" iyy="0.00002" iyz="0" izz="0.00002"/>
     </inertial>
   </link>
@@ -203,91 +209,117 @@
     <parent link="link5"/>
     <child link="gripper_base"/>
-    <origin xyz="0 0 0.1" rpy="0 0 0"/>
-  </joint>
-  <!-- Left Gripper Finger -->
-  <link name="gripper_left_finger">
-    <visual>
-      <origin xyz="0 0.015 0.025" rpy="0 0 0"/>
-      <geometry>
-        <box size="0.01 0.01 0.05"/>
-      </geometry>
-      <material name="black"/>
-    </visual>
-    <collision>
-      <origin xyz="0 0.015 0.025" rpy="0 0 0"/>
-      <geometry>
-        <box size="0.01 0.01 0.05"/>
-      </geometry>
-    </collision>
-    <inertial>
-      <origin xyz="0 0.015 0.025" rpy="0 0 0"/>
-      <mass value="0.01"/>
-      <inertia ixx="0.00001" ixy="0.0" ixz="0.0" iyy="0.00001" iyz="0.0" izz="0.00001"/>
+    <origin xyz="0 0 0.04" rpy="0 0 0"/>
+  </joint>
+  <!-- ===================== LEFT FINGER ===================== -->
+  <link name="gripper_left">
+    <visual>
+      <origin xyz="0 0 0.025" rpy="0 0 0"/>
+      <geometry>
+        <box size="0.01 0.015 0.05"/>
+      </geometry>
+      <material name="dark_grey"/>
+    </visual>
+    <collision>
+      <origin xyz="0 0 0.025" rpy="0 0 0"/>
+      <geometry>
+        <box size="0.01 0.015 0.05"/>
+      </geometry>
+    </collision>
+    <inertial>
+      <origin xyz="0 0 0.025" rpy="0 0 0"/>
+      <mass value="0.02"/>
+      <inertia ixx="0.000005" ixy="0" ixz="0" iyy="0.000005" iyz="0" izz="0.000002"/>
     </inertial>
   </link>
   <joint name="gripper_left_joint" type="prismatic">
     <parent link="gripper_base"/>
-    <child link="gripper_left_finger"/>
-    <origin xyz="0 0 0.04" rpy="0 0 0"/>
+    <child link="gripper_left"/>
+    <origin xyz="0 0.015 0.03" rpy="0 0 0"/>
     <axis xyz="0 1 0"/>
-    <limit lower="0" upper="0.03" effort="10" velocity="0.1"/>
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