Commit message: Adjust camera pose and spawn position for cube visibility

File: color_sorting_arm/urdf/arm.urdf.xacro (robot description, xacro)
@@ -286,5 +286,6 @@
     <parent link="gripper_base"/>
     <child link="camera_link"/>
-    <origin xyz="0.03 0 0.02" rpy="0 0 0"/>
+    <!-- Move camera forward/up and tilt it down to face the table -->
+    <origin xyz="0.07 0 0.05" rpy="0 -1.3 0"/>
   </joint>
   <!-- Camera Optical Frame -->

Commit message: Major fix: Camera position, cube locations, IK, and coordinate system corrections

File: color_sorting_arm/urdf/arm.urdf.xacro (robot description, xacro)
@@ -263,10 +263,10 @@
     <dynamics damping="0.3"/>
   </joint>
-  <!-- Camera Link -->
+  <!-- Camera Link - Mounted on link2 to look forward and down -->
   <link name="camera_link">
     <visual>
       <origin xyz="0 0 0" rpy="0 0 0"/>
       <geometry>
-        <box size="0.02 0.04 0.02"/>
+        <box size="0.03 0.05 0.03"/>
       </geometry>
       <material name="black"/>
@@ -275,5 +275,5 @@
       <origin xyz="0 0 0" rpy="0 0 0"/>
       <geometry>
-        <box size="0.02 0.04 0.02"/>
+        <box size="0.03 0.05 0.03"/>
       </geometry>
     </collision>
@@ -283,9 +283,9 @@
     </inertial>
   </link>
+  <!-- Camera mounted on link1 looking forward and down at table -->
   <joint name="camera_joint" type="fixed">
-    <parent link="gripper_base"/>
+    <parent link="link1"/>
     <child link="camera_link"/>
-    <!-- Move camera forward/up and tilt it down to face the table -->
-    <origin xyz="0.09 0 0.07" rpy="0 -1.45 0"/>
+    <origin xyz="0.08 0 0.15" rpy="0 0.6 0"/>
   </joint>
   <!-- Camera Optical Frame -->

Commit message: Major fix: longer arm, correct cube positions, high camera
URDF Changes:
- Link2: 0.15m (was 0.08m)
- Link3: 0.13m (was 0.07m)
- Link4: 0.08m (was 0.05m)
- Total reach now ~0.5m

World Changes:
- Camera on tall stand at 1.4m height, far behind robot
- Camera looking straight down at table
- Cubes properly placed on table surface (z=0.725)
- Cubes spread across table in reachable positions
- Bins at far end of table

Test Script:
- Clear 10-step test sequence
- Tests all joints and gripper
- Visual confirmation arm is working

File: color_sorting_arm/urdf/arm.urdf.xacro (robot description, xacro)
@@ -22,20 +22,20 @@
   <link name="base_link">
     <visual>
-      <origin xyz="0 0 0.02" rpy="0 0 0"/>
-      <geometry>
-        <cylinder radius="0.06" length="0.04"/>
+      <origin xyz="0 0 0.025" rpy="0 0 0"/>
+      <geometry>
+        <cylinder radius="0.07" length="0.05"/>
       </geometry>
       <material name="dark_grey"/>
     </visual>
     <collision>
-      <origin xyz="0 0 0.02" rpy="0 0 0"/>
-      <geometry>
-        <cylinder radius="0.06" length="0.04"/>
-      </geometry>
-    </collision>
-    <inertial>
-      <origin xyz="0 0 0.02" rpy="0 0 0"/>
-      <mass value="1.0"/>
-      <inertia ixx="0.002" ixy="0" ixz="0" iyy="0.002" iyz="0" izz="0.002"/>
+      <origin xyz="0 0 0.025" rpy="0 0 0"/>
+      <geometry>
+        <cylinder radius="0.07" length="0.05"/>
+      </geometry>
+    </collision>
+    <inertial>
+      <origin xyz="0 0 0.025" rpy="0 0 0"/>
+      <mass value="1.5"/>
+      <inertia ixx="0.003" ixy="0" ixz="0" iyy="0.003" iyz="0" izz="0.003"/>
     </inertial>
   </link>
@@ -43,20 +43,20 @@
   <link name="link1">
     <visual>
-      <origin xyz="0 0 0.025" rpy="0 0 0"/>
-      <geometry>
-        <cylinder radius="0.035" length="0.05"/>
+      <origin xyz="0 0 0.03" rpy="0 0 0"/>
+      <geometry>
+        <cylinder radius="0.045" length="0.06"/>
       </geometry>
       <material name="orange"/>
     </visual>
     <collision>
-      <origin xyz="0 0 0.025" rpy="0 0 0"/>
-      <geometry>
-        <cylinder radius="0.035" length="0.05"/>
-      </geometry>
-    </collision>
-    <inertial>
-      <origin xyz="0 0 0.025" rpy="0 0 0"/>
-      <mass value="0.3"/>
-      <inertia ixx="0.0005" ixy="0" ixz="0" iyy="0.0005" iyz="0" izz="0.0003"/>
+      <origin xyz="0 0 0.03" rpy="0 0 0"/>
+      <geometry>
+        <cylinder radius="0.045" length="0.06"/>
+      </geometry>
+    </collision>
+    <inertial>
+      <origin xyz="0 0 0.03" rpy="0 0 0"/>
+      <mass value="0.4"/>
+      <inertia ixx="0.0008" ixy="0" ixz="0" iyy="0.0008" iyz="0" izz="0.0005"/>
     </inertial>
   </link>
@@ -64,28 +64,28 @@
     <parent link="base_link"/>
     <child link="link1"/>
-    <origin xyz="0 0 0.04" rpy="0 0 0"/>
+    <origin xyz="0 0 0.05" rpy="0 0 0"/>
     <axis xyz="0 0 1"/>
-    <limit lower="${-PI}" upper="${PI}" effort="30" velocity="1.5"/>
-    <dynamics damping="0.5" friction="0.1"/>
-  </joint>
-  <!-- ===================== LINK 2 - SHOULDER ===================== -->
+    <limit lower="${-PI}" upper="${PI}" effort="50" velocity="1.5"/>
+    <dynamics damping="0.7" friction="0.2"/>
+  </joint>
+  <!-- ===================== LINK 2 - SHOULDER (LONGER) ===================== -->
   <link name="link2">
     <visual>
-      <origin xyz="0 0 0.04" rpy="0 0 0"/>
-      <geometry>
-        <box size="0.03 0.03 0.08"/>
+      <origin xyz="0 0 0.075" rpy="0 0 0"/>
+      <geometry>
+        <box size="0.05 0.04 0.15"/>
       </geometry>
       <material name="blue"/>
     </visual>
     <collision>
-      <origin xyz="0 0 0.04" rpy="0 0 0"/>
-      <geometry>
-        <box size="0.03 0.03 0.08"/>
-      </geometry>
-    </collision>
-    <inertial>
-      <origin xyz="0 0 0.04" rpy="0 0 0"/>
-      <mass value="0.2"/>
-      <inertia ixx="0.0003" ixy="0" ixz="0" iyy="0.0003" iyz="0" izz="0.0001"/>
+      <origin xyz="0 0 0.075" rpy="0 0 0"/>
+      <geometry>
+        <box size="0.05 0.04 0.15"/>
+      </geometry>
+    </collision>
+    <inertial>
+      <origin xyz="0 0 0.075" rpy="0 0 0"/>
+      <mass value="0.35"/>
+      <inertia ixx="0.001" ixy="0" ixz="0" iyy="0.001" iyz="0" izz="0.0003"/>
     </inertial>
   </link>
@@ -93,28 +93,28 @@
     <parent link="link1"/>
     <child link="link2"/>
-    <origin xyz="0 0 0.05" rpy="0 0 0"/>
-    <axis xyz="0 1 0"/>
-    <limit lower="${-PI/2}" upper="${PI/2}" effort="30" velocity="1.5"/>
-    <dynamics damping="0.5" friction="0.1"/>
-  </joint>
-  <!-- ===================== LINK 3 - ELBOW ===================== -->
+    <origin xyz="0 0 0.06" rpy="0 0 0"/>
+    <axis xyz="0 1 0"/>
+    <limit lower="${-PI/2}" upper="${PI/2}" effort="50" velocity="1.5"/>
+    <dynamics damping="0.7" friction="0.2"/>
+  </joint>
+  <!-- ===================== LINK 3 - ELBOW (LONGER) ===================== -->
   <link name="link3">
     <visual>
-      <origin xyz="0 0 0.035" rpy="0 0 0"/>
-      <geometry>
-        <box size="0.025 0.025 0.07"/>
+      <origin xyz="0 0 0.065" rpy="0 0 0"/>
+      <geometry>
+        <box size="0.04 0.035 0.13"/>
       </geometry>
       <material name="white"/>
     </visual>
     <collision>
-      <origin xyz="0 0 0.035" rpy="0 0 0"/>
-      <geometry>
-        <box size="0.025 0.025 0.07"/>
-      </geometry>
-    </collision>
-    <inertial>
-      <origin xyz="0 0 0.035" rpy="0 0 0"/>
-      <mass value="0.15"/>
-      <inertia ixx="0.0002" ixy="0" ixz="0" iyy="0.0002" iyz="0" izz="0.00005"/>
+      <origin xyz="0 0 0.065" rpy="0 0 0"/>
+      <geometry>
+        <box size="0.04 0.035 0.13"/>
+      </geometry>
+    </collision>
+    <inertial>
+      <origin xyz="0 0 0.065" rpy="0 0 0"/>
+      <mass value="0.25"/>
+      <inertia ixx="0.0006" ixy="0" ixz="0" iyy="0.0006" iyz="0" izz="0.0001"/>
     </inertial>
   </link>
@@ -122,28 +122,28 @@
     <parent link="link2"/>
     <child link="link3"/>
-    <origin xyz="0 0 0.08" rpy="0 0 0"/>
-    <axis xyz="0 1 0"/>
-    <limit lower="${-2.5}" upper="${2.5}" effort="20" velocity="1.5"/>
-    <dynamics damping="0.3" friction="0.1"/>
+    <origin xyz="0 0 0.15" rpy="0 0 0"/>
+    <axis xyz="0 1 0"/>
+    <limit lower="${-2.5}" upper="${2.5}" effort="40" velocity="1.5"/>
+    <dynamics damping="0.5" friction="0.15"/>
   </joint>
   <!-- ===================== LINK 4 - WRIST ===================== -->
   <link name="link4">
     <visual>
-      <origin xyz="0 0 0.025" rpy="0 0 0"/>
-      <geometry>
-        <box size="0.02 0.02 0.05"/>
+      <origin xyz="0 0 0.04" rpy="0 0 0"/>
+      <geometry>
+        <box size="0.035 0.03 0.08"/>
       </geometry>
       <material name="blue"/>
     </visual>
     <collision>
-      <origin xyz="0 0 0.025" rpy="0 0 0"/>
-      <geometry>
-        <box size="0.02 0.02 0.05"/>
-      </geometry>
-    </collision>
-    <inertial>
-      <origin xyz="0 0 0.025" rpy="0 0 0"/>
-      <mass value="0.1"/>
-      <inertia ixx="0.0001" ixy="0" ixz="0" iyy="0.0001" iyz="0" izz="0.00005"/>
+      <origin xyz="0 0 0.04" rpy="0 0 0"/>
+      <geometry>
+        <box size="0.035 0.03 0.08"/>
+      </geometry>
+    </collision>
+    <inertial>
+      <origin xyz="0 0 0.04" rpy="0 0 0"/>
+      <mass value="0.15"/>
+      <inertia ixx="0.0002" ixy="0" ixz="0" iyy="0.0002" iyz="0" izz="0.00008"/>
     </inertial>
   </link>
@@ -151,28 +151,28 @@
     <parent link="link3"/>
     <child link="link4"/>
-    <origin xyz="0 0 0.07" rpy="0 0 0"/>
-    <axis xyz="0 1 0"/>
-    <limit lower="${-PI/2}" upper="${PI/2}" effort="10" velocity="2.0"/>
-    <dynamics damping="0.2" friction="0.05"/>
+    <origin xyz="0 0 0.13" rpy="0 0 0"/>
+    <axis xyz="0 1 0"/>
+    <limit lower="${-PI/2}" upper="${PI/2}" effort="20" velocity="2.0"/>
+    <dynamics damping="0.3" friction="0.1"/>
   </joint>
   <!-- ===================== LINK 5 - WRIST ROLL ===================== -->
   <link name="link5">
     <visual>
-      <origin xyz="0 0 0.015" rpy="0 0 0"/>
-      <geometry>
-        <cylinder radius="0.015" length="0.03"/>
+      <origin xyz="0 0 0.02" rpy="0 0 0"/>
+      <geometry>
+        <cylinder radius="0.02" length="0.04"/>
       </geometry>
       <material name="white"/>
     </visual>
     <collision>
-      <origin xyz="0 0 0.015" rpy="0 0 0"/>
-      <geometry>
-        <cylinder radius="0.015" length="0.03"/>
-      </geometry>
-    </collision>
-    <inertial>
-      <origin xyz="0 0 0.015" rpy="0 0 0"/>
-      <mass value="0.05"/>
-      <inertia ixx="0.00002" ixy="0" ixz="0" iyy="0.00002" iyz="0" izz="0.00001"/>
+      <origin xyz="0 0 0.02" rpy="0 0 0"/>
+      <geometry>
+        <cylinder radius="0.02" length="0.04"/>
+      </geometry>
+    </collision>
+    <inertial>
+      <origin xyz="0 0 0.02" rpy="0 0 0"/>
+      <mass value="0.08"/>
+      <inertia ixx="0.00004" ixy="0" ixz="0" iyy="0.00004" iyz="0" izz="0.00002"/>
     </inertial>
   </link>
@@ -180,28 +180,28 @@
     <parent link="link4"/>
     <child link="link5"/>
-    <origin xyz="0 0 0.05" rpy="0 0 0"/>
+    <origin xyz="0 0 0.08" rpy="0 0 0"/>
     <axis xyz="0 0 1"/>
-    <limit lower="${-PI}" upper="${PI}" effort="5" velocity="2.0"/>
-    <dynamics damping="0.1" friction="0.05"/>
+    <limit lower="${-PI}" upper="${PI}" effort="10" velocity="2.0"/>
+    <dynamics damping="0.2" friction="0.05"/>
   </joint>
   <!-- ===================== GRIPPER BASE ===================== -->
   <link name="gripper_base">
     <visual>
-      <origin xyz="0 0 0.01" rpy="0 0 0"/>
-      <geometry>
-        <box size="0.02 0.04 0.02"/>
+      <origin xyz="0 0 0.015" rpy="0 0 0"/>
+      <geometry>
+        <box size="0.03 0.06 0.03"/>
       </geometry>
       <material name="grey"/>
     </visual>
     <collision>
-      <origin xyz="0 0 0.01" rpy="0 0 0"/>
-      <geometry>
-        <box size="0.02 0.04 0.02"/>
-      </geometry>
-    </collision>
-    <inertial>
-      <origin xyz="0 0 0.01" rpy="0 0 0"/>
-      <mass value="0.03"/>
-      <inertia ixx="0.00001" ixy="0" ixz="0" iyy="0.00001" iyz="0" izz="0.00001"/>
+      <origin xyz="0 0 0.015" rpy="0 0 0"/>
+      <geometry>
+        <box size="0.03 0.06 0.03"/>
+      </geometry>
+    </collision>
+    <inertial>
+      <origin xyz="0 0 0.015" rpy="0 0 0"/>
+      <mass value="0.05"/>
+      <inertia ixx="0.00002" ixy="0" ixz="0" iyy="0.00002" iyz="0" izz="0.00002"/>
     </inertial>
   </link>
@@ -209,25 +209,25 @@
     <parent link="link5"/>
     <child link="gripper_base"/>
-    <origin xyz="0 0 0.03" rpy="0 0 0"/>
+    <origin xyz="0 0 0.04" rpy="0 0 0"/>
   </joint>
   <!-- ===================== LEFT FINGER ===================== -->
   <link name="gripper_left">
     <visual>
-      <origin xyz="0 0 0.02" rpy="0 0 0"/>
-      <geometry>
-        <box size="0.008 0.01 0.04"/>
+      <origin xyz="0 0 0.03" rpy="0 0 0"/>
+      <geometry>
+        <box size="0.01 0.015 0.06"/>
       </geometry>
       <material name="dark_grey"/>
     </visual>
     <collision>
-      <origin xyz="0 0 0.02" rpy="0 0 0"/>
-      <geometry>
-        <box size="0.008 0.01 0.04"/>
-      </geometry>
-    </collision>
-    <inertial>
-      <origin xyz="0 0 0.02" rpy="0 0 0"/>
-      <mass value="0.01"/>
-      <inertia ixx="0.000002" ixy="0" ixz="0" iyy="0.000002" iyz="0" izz="0.000001"/>
+      <origin xyz="0 0 0.03" rpy="0 0 0"/>
+      <geometry>
+        <box size="0.01 0.015 0.06"/>
+      </geometry>
+    </collision>
+    <inertial>
+      <origin xyz="0 0 0.03" rpy="0 0 0"/>
+      <mass value="0.02"/>
+      <inertia ixx="0.000005" ixy="0" ixz="0" iyy="0.000005" iyz="0" izz="0.000002"/>
     </inertial>
   </link>
@@ -235,7 +235,7 @@
     <parent link="gripper_base"/>
     <child link="gripper_left"/>
-    <origin xyz="0 0.012 0.02" rpy="0 0 0"/>
-    <axis xyz="0 1 0"/>
-    <limit lower="0" upper="0.015" effort="5" velocity="0.1"/>
+    <origin xyz="0 0.02 0.03" rpy="0 0 0"/>
+    <axis xyz="0 1 0"/>
+    <limit lower="0" upper="0.025" effort="10" velocity="0.2"/>
     <dynamics damping="0.5"/>
   </joint>
@@ -243,20 +243,20 @@
   <link name="gripper_right">
     <visual>
-      <origin xyz="0 0 0.02" rpy="0 0 0"/>
-      <geometry>
-        <box size="0.008 0.01 0.04"/>
+      <origin xyz="0 0 0.03" rpy="0 0 0"/>
+      <geometry>
+        <box size="0.01 0.015 0.06"/>
       </geometry>
       <material name="dark_grey"/>
     </visual>
     <collision>
-      <origin xyz="0 0 0.02" rpy="0 0 0"/>
-      <geometry>
-        <box size="0.008 0.01 0.04"/>
-      </geometry>
-    </collision>
-    <inertial>
-      <origin xyz="0 0 0.02" rpy="0 0 0"/>
-      <mass value="0.01"/>
-      <inertia ixx="0.000002" ixy="0" ixz="0" iyy="0.000002" iyz="0" izz="0.000001"/>
+      <origin xyz="0 0 0.03" rpy="0 0 0"/>
+      <geometry>
+        <box size="0.01 0.015 0.06"/>
+      </geometry>
+    </collision>
+    <inertial>
+      <origin xyz="0 0 0.03" rpy="0 0 0"/>
+      <mass value="0.02"/>
+      <inertia ixx="0.000005" ixy="0" ixz="0" iyy="0.000005" iyz="0" izz="0.000002"/>
     </inertial>
   </link>
@@ -264,7 +264,7 @@
     <parent link="gripper_base"/>
     <child link="gripper_right"/>
-    <origin xyz="0 -0.012 0.02" rpy="0 0 0"/>
+    <origin xyz="0 -0.02 0.03" rpy="0 0 0"/>
     <axis xyz="0 -1 0"/>
-    <limit lower="0" upper="0.015" effort="5" velocity="0.1"/>
+    <limit lower="0" upper="0.025" effort="10" velocity="0.2"/>
     <dynamics damping="0.5"/>
   </joint>
