Commit message: Increase arm reach and move cubes closer

File: urdf/arm.urdf.xacro (robot description, xacro)
@@ -37,9 +37,9 @@
     </inertial>
   </link>
-  <link name="link1">
-    <visual>
-      <origin xyz="0 0 0.03" rpy="0 0 0"/>
-      <geometry>
-        <cylinder radius="0.045" length="0.06"/>
+  <link name="link2">
+    <visual>
+      <origin xyz="0 0 0.125" rpy="0 0 0"/>
+      <geometry>
+        <cylinder radius="0.025" length="0.25"/>
       </geometry>
       <material name="orange"/>
@@ -80,7 +80,7 @@
     </collision>
     <inertial>
-      <origin xyz="0 0 0.075" rpy="0 0 0"/>
-      <mass value="0.35"/>
-      <inertia ixx="0.001" ixy="0" ixz="0" iyy="0.001" iyz="0" izz="0.0003"/>
+      <origin xyz="0 0 0.125" rpy="0 0 0"/>
+      <mass value="0.4"/>
+      <inertia ixx="0.00208" ixy="0" ixz="0" iyy="0.00208" iyz="0" izz="0.00025"/>
     </inertial>
   </link>
@@ -90,5 +90,5 @@
     <origin xyz="0 0 0.06" rpy="0 0 0"/>
     <axis xyz="0 1 0"/>
-    <limit lower="${-PI/2}" upper="${PI/2}" effort="50" velocity="1.5"/>
+    <limit lower="-2.0" upper="2.0" effort="15.0" velocity="1.0"/>
     <dynamics damping="0.7" friction="0.2"/>
   </joint>
@@ -116,7 +116,7 @@
     <parent link="link2"/>
     <child link="link3"/>
-    <origin xyz="0 0 0.15" rpy="0 0 0"/>
-    <axis xyz="0 1 0"/>
-    <limit lower="${-2.5}" upper="${2.5}" effort="40" velocity="1.5"/>
+    <origin xyz="0 0 0.25" rpy="0 0 0"/>
+    <axis xyz="0 1 0"/>
+    <limit lower="-2.5" upper="0.5" effort="15.0" velocity="1.0"/>
     <dynamics damping="0.5" friction="0.15"/>
   </joint>
@@ -144,14 +144,14 @@
     <parent link="link3"/>
     <child link="link4"/>
-    <origin xyz="0 0 0.13" rpy="0 0 0"/>
-    <axis xyz="0 1 0"/>
-    <limit lower="${-PI/2}" upper="${PI/2}" effort="20" velocity="2.0"/>
+    <origin xyz="0 0 0.20" rpy="0 0 0"/>
+    <axis xyz="0 1 0"/>
+    <limit lower="-2.0" upper="2.0" effort="8.0" velocity="1.0"/>
     <dynamics damping="0.3" friction="0.1"/>
   </joint>
-  <link name="link5">
-    <visual>
-      <origin xyz="0 0 0.02" rpy="0 0 0"/>
-      <geometry>
-        <cylinder radius="0.02" length="0.04"/>
+  <link name="link3">
+    <visual>
+      <origin xyz="0 0 0.10" rpy="0 0 0"/>
+      <geometry>
+        <cylinder radius="0.02" length="0.20"/>
       </geometry>
       <material name="white"/>

Commit message: Remove duplicate link2 definition

File: urdf/arm.urdf.xacro (robot description, xacro)
@@ -35,24 +35,4 @@
       <mass value="1.5"/>
       <inertia ixx="0.003" ixy="0" ixz="0" iyy="0.003" iyz="0" izz="0.003"/>
-    </inertial>
-  </link>
-  <link name="link2">
-    <visual>
-      <origin xyz="0 0 0.125" rpy="0 0 0"/>
-      <geometry>
-        <cylinder radius="0.025" length="0.25"/>
-      </geometry>
-      <material name="orange"/>
-    </visual>
-    <collision>
-      <origin xyz="0 0 0.03" rpy="0 0 0"/>
-      <geometry>
-        <cylinder radius="0.045" length="0.06"/>
-      </geometry>
-    </collision>
-    <inertial>
-      <origin xyz="0 0 0.03" rpy="0 0 0"/>
-      <mass value="0.4"/>
-      <inertia ixx="0.0008" ixy="0" ixz="0" iyy="0.0008" iyz="0" izz="0.0005"/>
     </inertial>
   </link>

Commit message: Fix all URDF duplicates and add missing links (link1, link5), reduce approach height to 0.05m

File: urdf/arm.urdf.xacro (robot description, xacro)
@@ -35,4 +35,24 @@
       <mass value="1.5"/>
       <inertia ixx="0.003" ixy="0" ixz="0" iyy="0.003" iyz="0" izz="0.003"/>
+    </inertial>
+  </link>
+  <link name="link1">
+    <visual>
+      <origin xyz="0 0 0.03" rpy="0 0 0"/>
+      <geometry>
+        <cylinder radius="0.04" length="0.06"/>
+      </geometry>
+      <material name="grey"/>
+    </visual>
+    <collision>
+      <origin xyz="0 0 0.03" rpy="0 0 0"/>
+      <geometry>
+        <cylinder radius="0.04" length="0.06"/>
+      </geometry>
+    </collision>
+    <inertial>
+      <origin xyz="0 0 0.03" rpy="0 0 0"/>
+      <mass value="0.5"/>
+      <inertia ixx="0.001" ixy="0" ixz="0" iyy="0.001" iyz="0" izz="0.0008"/>
     </inertial>
   </link>
@@ -129,9 +149,9 @@
     <dynamics damping="0.3" friction="0.1"/>
   </joint>
-  <link name="link3">
-    <visual>
-      <origin xyz="0 0 0.10" rpy="0 0 0"/>
-      <geometry>
-        <cylinder radius="0.02" length="0.20"/>
+  <link name="link5">
+    <visual>
+      <origin xyz="0 0 0.02" rpy="0 0 0"/>
+      <geometry>
+        <cylinder radius="0.02" length="0.04"/>
       </geometry>
       <material name="white"/>

Commit message: Raise base_link origin to z=0.025 to prevent collision with ground

File: urdf/arm.urdf.xacro (robot description, xacro)
@@ -21,5 +21,5 @@
     <parent link="world"/>
     <child link="base_link"/>
-    <origin xyz="0 0 0" rpy="0 0 0"/>
+    <origin xyz="0 0 0.025" rpy="0 0 0"/>
   </joint>
   <link name="base_link">

Commit message: Adjust robot spawn and base_link origin to prevent collisions

File: urdf/arm.urdf.xacro (robot description, xacro)
@@ -21,5 +21,5 @@
     <parent link="world"/>
     <child link="base_link"/>
-    <origin xyz="0 0 0.025" rpy="0 0 0"/>
+    <origin xyz="0 0 0" rpy="0 0 0"/>
   </joint>
   <link name="base_link">

Commit message: Shorten link1 to 0.04m and shift joint2 origin to 0.04

File: urdf/arm.urdf.xacro (robot description, xacro)
@@ -59,6 +59,6 @@
     <inertial>
       <origin xyz="0 0 0.02" rpy="0 0 0"/>
-      <mass value="0.3"/>
-      <inertia ixx="0.0006" ixy="0" ixz="0" iyy="0.0006" iyz="0" izz="0.0004"/>
+      <mass value="0.5"/>
+      <inertia ixx="0.001" ixy="0" ixz="0" iyy="0.001" iyz="0" izz="0.0008"/>
     </inertial>
   </link>
